File: NixCard.kicad_pcb (KiCad board)
At the start: 2 copper layers, 21.6 x 31.8 mm, 7 parts, among them P1 TSW-104-07-F-S, P2 TSW-104-07-F-S, U1 NPIC6C4894

Commit message: Update PCB
Parts:
- added REF***: OSHW-Logo_5.7x6mm_SilkScreen, Symbols:OSHW-Logo_5.7x6mm_SilkScreen, F.Cu at (141.1, 117.0)
Other:
- board text added: "REV A 2016 DEC 24"
- board text added: "github.com/RobertBaruch/NixCard"

Commit message: Updated PCB
Parts:
- added REF**: MountingHole_2.2mm_M2, Mounting_Holes:MountingHole_2.2mm_M2, F.Cu at (156.7, 117.9)
- added REF**: MountingHole_2.2mm_M2, Mounting_Holes:MountingHole_2.2mm_M2, F.Cu at (156.7, 91.7)
- added REF**: MountingHole_2.2mm_M2, Mounting_Holes:MountingHole_2.2mm_M2, F.Cu at (140.5, 91.7)
- added REF**: MountingHole_2.2mm_M2, Mounting_Holes:MountingHole_2.2mm_M2, F.Cu at (140.5, 117.9)
- REF***: moved to B.Cu
- moved R1 18.5 mm to (140.5, 112.8), turned to 0 degrees
- moved REF*** 11.8 mm to (148.6, 108.0), turned to 180 degrees
- moved P1 0.63 mm to (152.4, 117.5)
- moved P2 0.63 mm to (152.4, 92.1)
Routing:
- net VAA: track 3.44 -> 24.8 mm
- net Net-(N1-PadA): track 21.4 -> 3.11 mm
- net /LE: track 21.4 -> 15.3 mm, vias 0 -> 1
- net /DIN: track 13.6 -> 16.6 mm
- net /CP: track 14.0 -> 16.7 mm
- net /DOUT: track 26.0 -> 28.2 mm
- net GNDREF: track 7.01 -> 4.97 mm
- net +5V: track 20.0 -> 21.9 mm
- net /OE: track 15.8 -> 17.6 mm
- net Net-(N1-Pad1): track 12.2 -> 12.7 mm
Other:
- board text added: "REV B 2017 JAN 15"
- board text added: "THIS END UP"
- board text added: "USE 2-56 OR M2 SCREWS"
- board text removed: "REV A 2016 DEC 24"
